File: tester/mcu.kicad_sch (KiCad schematic)
At the start: 38 parts, among them J201 PWR, J202 SWD, Q201 SI2301CDS-T1-GE3, SW201 Reset, U201 AMS1117-3.3, U202 STM32F103C8Tx, U203 M24C64-RMN, U204 M24C64-RMN, Y201 8MHz, Y202 32k

Commit message: Use correct footprint for D201
Signed-off-by: Benedikt Spranger <b.spranger@linutronix.de>
Parts:
- D201: footprint Diode_SMD:D_SOD-123 -> Diode_SMD:D_SOD-323
Changed lines of the file:
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@@
 			)
 		)
-		(property "Footprint" "Diode_SMD:D_SOD-123"
+		(property "Footprint" "Diode_SMD:D_SOD-323"
 			(at 109.855 31.75 0)
 			(hide yes)
