File: tester/tester.kicad_pcb (KiCad board)
At the start: 4 copper layers, 150 x 120 mm, 139 parts, among them J101 X1, J102 X3, J103 X2, J201 PWR, J202 SWD, J306 DISP, J307 SD-Card, J401 USB_B_Micro, Q201 SI2301CDS-T1-GE3, SW201 Reset, SW301 SW_Push, SW302 SW_Push, SW303 SW_Push, SW304 SW_Push, SW305 SW_Push, U101 PCA9539xPW, U102 PCA9539xPW, U201 AMS1117-3.3, U202 STM32F103C8Tx, U203 M24C64-RMN, U204 M24C64-RMN, U401 USBLC6-2SC6, U402 XC6206P332MR, U403 CH340N, Y201 8MHz, Y202 32k

Commit message: Use correct footprint for D201
Signed-off-by: Benedikt Spranger <b.spranger@linutronix.de>
Parts:
- D201: footprint Diode_SMD:D_SOD-123 -> Diode_SMD:D_SOD-323
Changed lines of the file:
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@@
 				(name "A")
 				(pins "7" "44" "5" "6" "2" "3" "4" "18" "19" "20" "39" "40" "41" "42"
-					"43" "45" "46" "21" "22" "25" "26" "27" "28" "1" "24" "36" "23" "35"
-					"47" "48" "8" "9" "10" "11" "12" "13" "14" "15" "16" "17" "29" "30"
+					"43" "45" "46" "21" "22" "25" "26" "27" "28" "1" "24" "36" "47" "23"
+					"35" "48" "8" "9" "10" "11" "12" "13" "14" "15" "16" "17" "29" "30"
 					"31" "32" "33" "34" "37" "38"
 				)
@@
 		)
 	)
-	(footprint "Diode_SMD:D_SOD-123"
+	(footprint "Diode_SMD:D_SOD-323"
 		(layer "F.Cu")
 		(at 181.381636 89.25)
-		(descr "SOD-123")
-		(tags "SOD-123")
+		(descr "SOD-323")
+		(tags "SOD-323")
 		(property "Reference" "D201"
-			(at 0 -2 0)
+			(at 0 -1.85 0)
 			(layer "F.SilkS")
 			(effects
@@
 		)
 		(property "Value" "1N4148WS"
-			(at 0 2.1 0)
+			(at 0.1 1.9 0)
 			(layer "F.Fab")
 			(effects
@@
 		(duplicate_pad_numbers_are_jumpers no)
 		(fp_line
-			(start -2.36 -1)
-			(end -2.36 1)
+			(start -1.61 -0.85)
+			(end -1.61 0.85)
 			(stroke
 				(width 0.12)
@@
 		)
 		(fp_line
-			(start -2.36 -1)
-			(end 1.65 -1)
+			(start -1.61 -0.85)
+			(end 1.05 -0.85)
 			(stroke
 				(width 0.12)
@@
 		)
 		(fp_line
-			(start -2.36 1)
-			(end 1.65 1)
+			(start -1.61 0.85)
+			(end 1.05 0.85)
 			(stroke
 				(width 0.12)
@@
 		)
 		(fp_line
-			(start -2.35 -1.15)
-			(end -2.35 1.15)
+			(start -1.6 -0.95)
+			(end -1.6 0.95)
 			(stroke
 				(width 0.05)
@@
 		)
 		(fp_line
-			(start -2.35 -1.15)
-			(end 2.35 -1.15)
+			(start -1.6 -0.95)
+			(end 1.6 -0.95)
 			(stroke
 				(width 0.05)
@@
 		)
 		(fp_line
-			(start 2.35 -1.15)
-			(end 2.35 1.15)
+			(start -1.6 0.95)
+			(end 1.6 0.95)
 			(stroke
 				(width 0.05)
@@
 		)
 		(fp_line
-			(start 2.35 1.15)
-			(end -2.35 1.15)
+			(start 1.6 -0.95)
+			(end 1.6 0.95)
 			(stroke
 				(width 0.05)
@@
 		)
 		(fp_line
-			(start -1.4 -0.9)
-			(end 1.4 -0.9)
+			(start -0.9 -0.7)
+			(end 0.9 -0.7)
 			(stroke
 				(width 0.1)
@@
 		)
 		(fp_line
-			(start -1.4 0.9)
-			(end -1.4 -0.9)
+			(start -0.9 0.7)
+			(end -0.9 -0.7)
 			(stroke
 				(width 0.1)
@@
 		)
 		(fp_line
-			(start -0.75 0)
-			(end -0.35 0)
+			(start -0.3 -0.35)
+			(end -0.3 0.35)
 			(stroke
 				(width 0.1)
@@
 		)
 		(fp_line
-			(start -0.35 0)
-			(end -0.35 -0.55)
+			(start -0.3 0)
+			(end -0.5 0)
 			(stroke
 				(width 0.1)
@@
 		)
 		(fp_line
-			(start -0.35 0)
-			(end -0.35 0.55)
+			(start -0.3 0)
+			(end 0.2 -0.35)
 			(stroke
 				(width 0.1)
@@
 		)
 		(fp_line
-			(start -0.35 0)
-			(end 0.25 -0.4)
+			(start 0.2 -0.35)
+			(end 0.2 0.35)
 			(stroke
 				(width 0.1)
@@
 		)
 		(fp_line
-			(start 0.25 -0.4)
-			(end 0.25 0.4)
+			(start 0.2 0)
+			(end 0.45 0)
 			(stroke
 				(width 0.1)
@@
 		)
 		(fp_line
-			(start 0.25 0)
-			(end 0.75 0)
+			(start 0.2 0.35)
+			(end -0.3 0)
 			(stroke
 				(width 0.1)
@@
 		)
 		(fp_line
-			(start 0.25 0.4)
-			(end -0.35 0)
+			(start 0.9 -0.7)
+			(end 0.9 0.7)
 			(stroke
 				(width 0.1)
@@
 		)
 		(fp_line
-			(start 1.4 -0.9)
-			(end 1.4 0.9)
-			(stroke
-				(width 0.1)
-				(type solid)
-			)
-			(layer "F.Fab")
-		)
-		(fp_line
-			(start 1.4 0.9)
-			(end -1.4 0.9)
+			(start 0.9 0.7)
+			(end -0.9 0.7)
 			(stroke
 				(width 0.1)
@@
 		)
 		(fp_text user "${REFERENCE}"
-			(at 0 -2 0)
+			(at 0 -1.85 0)
 			(layer "F.Fab")
 			(effects
@@
 		)
 		(pad "1" smd roundrect
-			(at -1.65 0)
-			(size 0.9 1.2)
+			(at -1.05 0)
+			(size 0.6 0.45)
 			(layers "F.Cu" "F.Mask" "F.Paste")
 			(roundrect_rratio 0.25)
@@
 		)
 		(pad "2" smd roundrect
-			(at 1.65 0)
-			(size 0.9 1.2)
+			(at 1.05 0)
+			(size 0.6 0.45)
 			(layers "F.Cu" "F.Mask" "F.Paste")
 			(roundrect_rratio 0.25)
@@
 		)
 		(embedded_fonts no)
-		(model "${KICAD10_3DMODEL_DIR}/Diode_SMD.3dshapes/D_SOD-123.step"
+		(model "${KICAD10_3DMODEL_DIR}/Diode_SMD.3dshapes/D_SOD-323.step"
 			(offset
 				(xyz 0 0 0)
