File: tester/serial.kicad_sch (KiCad schematic)
At the start: 11 parts, among them J401 USB_B_Micro, U401 USBLC6-2SC6, U402 XC6206P332MR, U403 CH340N

Commit message: Add automation for tester
Signed-off-by: Benedikt Spranger <b.spranger@linutronix.de>
Other:
- company: Eurovibes Benedikt Spranger -> Benedikt Spranger
- title: DCC Licht -> rack-ser-adapter-tester
Changed lines of the file:
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@@
 	(paper "A4")
 	(title_block
-		(title "DCC Licht")
-		(date "2025-01-22")
+		(title "rack-ser-adapter-tester")
+		(date "2026-09-15")
 		(rev "v0.1")
-		(company "Eurovibes Benedikt Spranger")
+		(company "Benedikt Spranger")
 		(comment 1 "SPDX-License-Identifier: CERN-OHL-S-2.0")
 		(comment 2 "https://ohwr.org/cern_ohl_s_v2.txt")

Commit message: Fix USB connector part information
Signed-off-by: Benedikt Spranger <b.spranger@linutronix.de>
Parts:
- J401: LCSC# C132563 -> C132562; MF (none) -> Amphenol ICC; MP (none) -> 10118193-0001LF; mpn 10118194-0001LF -> 10118193-0001LF
Changed lines of the file:
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@@
 			)
 		)
-		(property "LCSC#" "C132563"
+		(property "LCSC#" "C132562"
 			(at 125.73 67.31 0)
 			(hide yes)
@@
 			)
 		)
-		(property "mpn" "10118194-0001LF"
+		(property "mpn" "10118193-0001LF"
 			(at 125.73 67.31 0)
 			(hide yes)
+			(show_name no)
+			(do_not_autoplace no)
+			(effects
+				(font
+					(size 1.27 1.27)
+				)
+			)
+		)
+		(property "MF" "Amphenol ICC"
+			(at 125.73 67.31 0)
+			(hide yes)
+			(show_name no)
+			(do_not_autoplace no)
+			(effects
+				(font
+					(size 1.27 1.27)
+				)
+			)
+		)
+		(property "MP" "10118193-0001LF"
+			(at 125.73 67.31 0)
+			(hide yes)

Commit message: Enable CH340N 3.3V operation
Signed-off-by: Benedikt Spranger <b.spranger@linutronix.de>
Connections:
- net at C402.1, C403.1, D401.2 (A)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: now also C404.1, U403.8 (V3)
Changed lines of the file:
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@@
+	)
+	(junction
+		(at 203.2 62.23)
+		(diameter 0)
+		(color 0 0 0 0)
 	)
 	(junction
@@
 	(junction
 		(at 196.85 31.75)
+		(diameter 0)
+		(color 0 0 0 0)
+	)
+	(junction
+		(at 215.9 54.61)
 		(diameter 0)
 		(color 0 0 0 0)
@@
 	(wire
 		(pts
+			(xy 203.2 62.23) (xy 203.2 54.61)
+		)
+		(stroke
+			(width 0)
+			(type default)
+		)
+	)
+	(wire
+		(pts
 			(xy 203.2 80.01) (xy 203.2 82.55)
 		)
@@
 	(wire
 		(pts
+			(xy 215.9 54.61) (xy 215.9 31.75)
+		)
+		(stroke
+			(width 0)
+			(type default)
+		)
+	)
+	(wire
+		(pts
 			(xy 215.9 31.75) (xy 196.85 31.75)
 		)
@@
 	(wire
 		(pts
-			(xy 215.9 57.15) (xy 215.9 31.75)
-		)
-		(stroke
+			(xy 203.2 54.61) (xy 215.9 54.61)
+		)
+		(stroke
+			(width 0)
+			(type default)
+		)
+	)
+	(wire
+		(pts
+			(xy 215.9 57.15) (xy 215.9 54.61)
+		)
+		(stroke

Commit message: Add LDO recommended tantalum capacitor
Signed-off-by: Benedikt Spranger <b.spranger@linutronix.de>
Parts:
- FB401: Long Description (none) -> -55℃~+125℃ 1 200mA 450mΩ 600Ω@100MHz ±25% 0603 Ferrite Bead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; MF (none) -> Sunlord; MP (none) -> GZ1608D601TF
Changed lines of the file:
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@@
+			)
+		)
+		(property "Long Description" "-55℃~+125℃ 1 200mA 450mΩ 600Ω@100MHz ±25% 0603 Ferrite Beads ROHS"
+			(at 123.19 82.55 0)
+			(hide yes)
+			(show_name no)
+			(do_not_autoplace no)
+			(effects
+				(font
+					(size 1.27 1.27)
+				)
+			)
+		)
+		(property "MF" "Sunlord"
+			(at 123.19 82.55 0)
+			(hide yes)
+			(show_name no)
+			(do_not_autoplace no)
+			(effects
+				(font
+					(size 1.27 1.27)
+				)
+			)
+		)
+		(property "MP" "GZ1608D601TF"
+			(at 123.19 82.55 0)
+			(hide yes)
+			(show_name no)
+			(do_not_autoplace no)
+			(effects
+				(font
+					(size 1.27 1.27)
+				)
 			)
 		)
