File: invers/rack-ser-adapter-inv.kicad_pcb (KiCad board)
At the start: 2 copper layers, 34 x 71 mm, 8 parts, among them J1 RS-232, J2 RJ45_Shielded, J3 RS-232, J4 RJ45_Shielded

Commit message: Add connector marker
Signed-off-by: Benedikt Spranger <b.spranger@linutronix.de>
Other:
- board text added: "♀"
- board text added: "♂"
Changed lines of the file:
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@@
+		)
+	)
+	(gr_text "♀"
+		(at 118 76 0)
+		(layer "F.Cu")
+		(effects
+			(font
+				(face "DejaVu Sans")
+				(size 1.5 1.5)
+				(thickness 0.3)
+				(bold yes)
+			)
+			(justify left bottom)
+		)
+		(render_cache "♀" 0
+			(polygon
+				(pts
+					(xy 118.885392 74.220861) (xy 118.992947 74.252559) (xy 119.091935 74.305113) (xy 119.183997 74.380109)
+					(xy 119.260524 74.47063) (xy 119.314155 74.568699) (xy 119.346552 74.67604) (xy 119.357654 74.795109)
+					(xy 119.350426 74.891648) (xy 119.329428 74.979027) (xy 119.29512 75.058776) (xy 119.247183 75.132109)
+					(xy 119.184547 75.199849) (xy 119.111192 75.258067) (xy 119.033389 75.301543) (xy 118.950297 75.331237)
+					(xy 118.860772 75.347403) (xy 118.860772 75.617963) (xy 119.139484 75.617963) (xy 119.139484 75.745)
+					(xy 118.860772 75.745) (xy 118.860772 76.008324) (xy 118.676308 76.008324) (xy 118.676308 75.745)
+					(xy 118.397596 75.745) (xy 118.397596 75.617963) (xy 118.676308 75.617963) (xy 118.676308 75.346395)
+					(xy 118.586196 75.330626) (xy 118.502947 75.301202) (xy 118.425354 75.257923) (xy 118.352534 75.199849)
+					(xy 118.289807 75.131694) (xy 118.241833 75.058092) (xy 118.207526 74.978231) (xy 118.186549 74.890919)
+					(xy 118.179335 74.794651) (xy 118.363799 74.794651) (xy 118.37145 74.876161) (xy 118.393641 74.948556)
+					(xy 118.430182 75.013681) (xy 118.482135 75.072813) (xy 118.544547 75.121367) (xy 118.612014 75.155599)
+					(xy 118.685652 75.176344) (xy 118.766983 75.183455) (xy 118.848297 75.176365) (xy 118.922215 75.155649)
+					(xy 118.990215 75.121416) (xy 119.053388 75.072813) (xy 119.106094 75.013586) (xy 119.143101 74.94843)
+					(xy 119.165548 74.876072) (xy 119.173281 74.794651) (xy 119.165633 74.713225) (xy 119.143297 74.63972)
+					(xy 119.106278 74.572457) (xy 119.053388 74.51026) (xy 118.98985 74.458719) (xy 118.921746 74.422638)
+					(xy 118.847972 74.400903) (xy 118.766983 74.393482) (xy 118.685982 74.400924) (xy 118.612486 74.422688)
+					(xy 118.544914 74.458767) (xy 118.482135 74.51026) (xy 118.429996 74.572363) (xy 118.393445 74.639598)
+					(xy 118.371365 74.713139) (xy 118.363799 74.794651) (xy 118.179335 74.794651) (xy 118.190346 74.675739)
+					(xy 118.222474 74.568513) (xy 118.275635 74.470541) (xy 118.351434 74.380109) (xy 118.442782 74.305159)
+					(xy 118.541271 74.252606) (xy 118.648562 74.220881) (xy 118.766983 74.210025)
+				)
+			)
+		)
+	)
+	(gr_text "♂"
+		(at 118 112 0)
+		(layer "F.Cu")
+		(effects
+			(font
+				(face "DejaVu Sans")
+				(size 1.5 1.5)
+				(thickness 0.3)
+				(bold yes)
+			)
+			(justify left bottom)
+		)
+		(render_cache "♂" 0
+			(polygon
+				(pts
+					(xy 119.742978 110.737773) (xy 119.596432 110.884227) (xy 119.596432 110.502109) (xy 119.22961 110.858673)
+					(xy 119.279717 110.936277) (xy 119.315336 111.019242) (xy 119.336975 111.108678) (xy 119.344373 111.205986)
+					(xy 119.333545 111.321521) (xy 119.301931 111.425776) (xy 119.249553 111.521133) (xy 119.174747 111.609262)
+					(xy 119.084996 111.681786) (xy 118.987181 111.732941) (xy 118.879567 111.763999) (xy 118.759747 111.774675)
+					(xy 118.639862 111.764229) (xy 118.531365 111.733766) (xy 118.432016 111.683518) (xy 118.340169 111.612284)
+					(xy 118.276969 111.543447) (xy 118.228698 111.469382) (xy 118.194231 111.389295) (xy 118.173189 111.302019)
+					(xy 118.165963 111.206078) (xy 118.350427 111.206078) (xy 118.358084 111.287832) (xy 118.380287 111.360393)
+					(xy 118.41683 111.425618) (xy 118.468763 111.484789) (xy 118.531175 111.533344) (xy 118.598642 111.567576)
+					(xy 118.67228 111.58832) (xy 118.753611 111.595431) (xy 118.834925 111.588341) (xy 118.908843 111.567626)
+					(xy 118.976843 111.533393) (xy 119.040016 111.484789) (xy 119.092701 111.425522) (xy 119.12971 111.360267)
+					(xy 119.152169 111.287742) (xy 119.159909 111.206078) (xy 119.152252 111.124409) (xy 119.129903 111.050754)
+					(xy 119.092882 110.983421) (xy 119.040016 110.921229) (xy 118.976472 110.869644) (xy 118.908367 110.833535)
+					(xy 118.834595 110.811785) (xy 118.753611 110.804359) (xy 118.672614 110.811806) (xy 118.599121 110.833586)
+					(xy 118.531547 110.869692) (xy 118.468763 110.921229) (xy 118.416647 110.983327) (xy 118.380094 111.050631)
+					(xy 118.358 111.124323) (xy 118.350427 111.206078) (xy 118.165963 111.206078) (xy 118.177149 111.087746)
+					(xy 118.209942 110.979986) (xy 118.264508 110.880455) (xy 118.342733 110.787506) (xy 118.417653 110.723558)
+					(xy 118.495371 110.676066) (xy 118.576626 110.643561) (xy 118.662459 110.625329) (xy 118.75416 110.621452)
+					(xy 118.873052 110.633367) (xy 118.968225 110.657522) (xy 119.043914 110.69194) (xy 119.10358 110.735666)
+					(xy 119.473517 110.379102) (xy 119.093322 110.379102) (xy 119.236754 110.233564) (xy 119.742978 110.233564)
+				)
+			)
 		)
 	)
