File: norm/rack-ser-adapter.kicad_pcb (KiCad board)
At the start: 2 copper layers, 34 x 71 mm, 8 parts, among them J1 RS-232, J2 RJ45_Shielded, J3 RS-232, J4 RJ45_Shielded

Commit message: Add connector marker
Signed-off-by: Benedikt Spranger <b.spranger@linutronix.de>
Other:
- board text added: "♀"
- board text added: "♂"
Changed lines of the file:
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@@
+		)
+	)
+	(gr_text "♂"
+		(at 118 76 0)
+		(layer "F.Cu")
+		(effects
+			(font
+				(face "DejaVu Sans")
+				(size 1.5 1.5)
+				(thickness 0.3)
+				(bold yes)
+			)
+			(justify left bottom)
+		)
+		(render_cache "♂" 0
+			(polygon
+				(pts
+					(xy 119.742978 74.737773) (xy 119.596432 74.884227) (xy 119.596432 74.502109) (xy 119.22961 74.858673)
+					(xy 119.279717 74.936277) (xy 119.315336 75.019242) (xy 119.336975 75.108678) (xy 119.344373 75.205986)
+					(xy 119.333545 75.321521) (xy 119.301931 75.425776) (xy 119.249553 75.521133) (xy 119.174747 75.609262)
+					(xy 119.084996 75.681786) (xy 118.987181 75.732941) (xy 118.879567 75.763999) (xy 118.759747 75.774675)
+					(xy 118.639862 75.764229) (xy 118.531365 75.733766) (xy 118.432016 75.683518) (xy 118.340169 75.612284)
+					(xy 118.276969 75.543447) (xy 118.228698 75.469382) (xy 118.194231 75.389295) (xy 118.173189 75.302019)
+					(xy 118.165963 75.206078) (xy 118.350427 75.206078) (xy 118.358084 75.287832) (xy 118.380287 75.360393)
+					(xy 118.41683 75.425618) (xy 118.468763 75.484789) (xy 118.531175 75.533344) (xy 118.598642 75.567576)
+					(xy 118.67228 75.58832) (xy 118.753611 75.595431) (xy 118.834925 75.588341) (xy 118.908843 75.567626)
+					(xy 118.976843 75.533393) (xy 119.040016 75.484789) (xy 119.092701 75.425522) (xy 119.12971 75.360267)
+					(xy 119.152169 75.287742) (xy 119.159909 75.206078) (xy 119.152252 75.124409) (xy 119.129903 75.050754)
+					(xy 119.092882 74.983421) (xy 119.040016 74.921229) (xy 118.976472 74.869644) (xy 118.908367 74.833535)
+					(xy 118.834595 74.811785) (xy 118.753611 74.804359) (xy 118.672614 74.811806) (xy 118.599121 74.833586)
+					(xy 118.531547 74.869692) (xy 118.468763 74.921229) (xy 118.416647 74.983327) (xy 118.380094 75.050631)
+					(xy 118.358 75.124323) (xy 118.350427 75.206078) (xy 118.165963 75.206078) (xy 118.177149 75.087746)
+					(xy 118.209942 74.979986) (xy 118.264508 74.880455) (xy 118.342733 74.787506) (xy 118.417653 74.723558)
+					(xy 118.495371 74.676066) (xy 118.576626 74.643561) (xy 118.662459 74.625329) (xy 118.75416 74.621452)
+					(xy 118.873052 74.633367) (xy 118.968225 74.657522) (xy 119.043914 74.69194) (xy 119.10358 74.735666)
+					(xy 119.473517 74.379102) (xy 119.093322 74.379102) (xy 119.236754 74.233564) (xy 119.742978 74.233564)
+				)
+			)
+		)
+	)
+	(gr_text "♀"
+		(at 118 112 0)
+		(layer "F.Cu")
+		(effects
+			(font
+				(face "DejaVu Sans")
+				(size 1.5 1.5)
+				(thickness 0.3)
+				(bold yes)
+			)
+			(justify left bottom)
+		)
+		(render_cache "♀" 0
+			(polygon
+				(pts
+					(xy 118.885392 110.220861) (xy 118.992947 110.252559) (xy 119.091935 110.305113) (xy 119.183997 110.380109)
+					(xy 119.260524 110.47063) (xy 119.314155 110.568699) (xy 119.346552 110.67604) (xy 119.357654 110.795109)
+					(xy 119.350426 110.891648) (xy 119.329428 110.979027) (xy 119.29512 111.058776) (xy 119.247183 111.132109)
+					(xy 119.184547 111.199849) (xy 119.111192 111.258067) (xy 119.033389 111.301543) (xy 118.950297 111.331237)
+					(xy 118.860772 111.347403) (xy 118.860772 111.617963) (xy 119.139484 111.617963) (xy 119.139484 111.745)
+					(xy 118.860772 111.745) (xy 118.860772 112.008324) (xy 118.676308 112.008324) (xy 118.676308 111.745)
+					(xy 118.397596 111.745) (xy 118.397596 111.617963) (xy 118.676308 111.617963) (xy 118.676308 111.346395)
+					(xy 118.586196 111.330626) (xy 118.502947 111.301202) (xy 118.425354 111.257923) (xy 118.352534 111.199849)
+					(xy 118.289807 111.131694) (xy 118.241833 111.058092) (xy 118.207526 110.978231) (xy 118.186549 110.890919)
+					(xy 118.179335 110.794651) (xy 118.363799 110.794651) (xy 118.37145 110.876161) (xy 118.393641 110.948556)
+					(xy 118.430182 111.013681) (xy 118.482135 111.072813) (xy 118.544547 111.121367) (xy 118.612014 111.155599)
+					(xy 118.685652 111.176344) (xy 118.766983 111.183455) (xy 118.848297 111.176365) (xy 118.922215 111.155649)
+					(xy 118.990215 111.121416) (xy 119.053388 111.072813) (xy 119.106094 111.013586) (xy 119.143101 110.94843)
+					(xy 119.165548 110.876072) (xy 119.173281 110.794651) (xy 119.165633 110.713225) (xy 119.143297 110.63972)
+					(xy 119.106278 110.572457) (xy 119.053388 110.51026) (xy 118.98985 110.458719) (xy 118.921746 110.422638)
+					(xy 118.847972 110.400903) (xy 118.766983 110.393482) (xy 118.685982 110.400924) (xy 118.612486 110.422688)
+					(xy 118.544914 110.458767) (xy 118.482135 110.51026) (xy 118.429996 110.572363) (xy 118.393445 110.639598)
+					(xy 118.371365 110.713139) (xy 118.363799 110.794651) (xy 118.179335 110.794651) (xy 118.190346 110.675739)
+					(xy 118.222474 110.568513) (xy 118.275635 110.470541) (xy 118.351434 110.380109) (xy 118.442782 110.305159)
+					(xy 118.541271 110.252606) (xy 118.648562 110.220881) (xy 118.766983 110.210025)
+				)
+			)
 		)
 	)
